File: main.kicad_pcb (KiCad board)
At the start: 2 copper layers, 256 x 88.5 mm, 92 parts, among them SW1 SW_PUSH, SW10 SW_PUSH, SW11 SW_PUSH, SW12 SW_PUSH, SW13 SW_PUSH, SW14 SW_PUSH, SW15 SW_PUSH, SW16 SW_PUSH, SW17 SW_PUSH, SW18 SW_PUSH, SW19 SW_PUSH, SW2 SW_PUSH, SW20 SW_PUSH, SW21 SW_PUSH, SW22 SW_PUSH, SW23 SW_PUSH, SW24 SW_PUSH, SW25 SW_PUSH, SW26 SW_PUSH, SW27 SW_PUSH, SW28 SW_PUSH, SW29 SW_PUSH, SW3 SW_PUSH, SW30 SW_PUSH, SW31 SW_PUSH, SW32 SW_PUSH, SW33 SW_PUSH, SW34 SW_PUSH, SW35 SW_PUSH, SW36 SW_PUSH, SW37 SW_PUSH, SW38 SW_PUSH, SW39 SW_PUSH, SW4 SW_PUSH, SW40 SW_PUSH, SW41 SW_PUSH, SW42 SW_PUSH, SW43 SW_PUSH, SW44 SW_PUSH, SW5 SW_PUSH, SW6 SW_PUSH, SW7 SW_PUSH, SW8 SW_PUSH, SW9 SW_PUSH, U1 RP2040_ZERO

Commit message: WIP
Parts:
- moved D34 4.38 mm to (221.6, 91.2), turned to -168 degrees
- moved D22 3.35 mm to (228.6, 71.0), turned to -168 degrees
- moved D20 2.46 mm to (191.0, 79.0), turned to -168 degrees
- moved D21 2.40 mm to (208.5, 75.1), turned to -168 degrees
- moved D9 2.35 mm to (208.6, 57.0), turned to -168 degrees
- moved D35 2.35 mm to (241.6, 90.7)
- moved D36 2.35 mm to (259.6, 90.7)
- moved D10 2.33 mm to (226.3, 53.2), turned to -168 degrees
- moved D33 2.03 mm to (203.6, 94.7), turned to -168 degrees
- moved D8 2.01 mm to (191.1, 60.7), turned to -168 degrees
- moved D32 1.91 mm to (186.0, 98.6), turned to -168 degrees
- moved D41 1.75 mm to (163.6, 121.7), turned to -168 degrees
- moved D42 1.70 mm to (181.2, 118.0), turned to -168 degrees
- moved D7 1.66 mm to (173.3, 64.5), turned to -168 degrees
- moved D44 1.63 mm to (216.5, 110.5), turned to -168 degrees
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Routing:
- net /row2: track 37.5 -> 459.7 mm, vias 3 -> 13
- net /row3: track 26.8 -> 316.6 mm, vias 3 -> 9
- net /row1: track 238.8 -> 456.1 mm, vias 8 -> 13
- net /row0: track 249.8 -> 464.6 mm, vias 8 -> 13
- net /col4: track 131.9 -> 136.9 mm
- net Net-(D37-A): track 0.00 -> 3.95 mm
- net /col3: track 144.8 -> 148.4 mm
- net Net-(D22-A): track 6.89 -> 3.48 mm
- net Net-(D34-A): track 6.41 -> 3.55 mm
- net Net-(D21-A): track 4.85 -> 2.60 mm
- net Net-(D27-A): track 4.56 -> 2.43 mm
- net Net-(D9-A): track 5.01 -> 2.94 mm
- net Net-(D33-A): track 4.55 -> 2.51 mm
- net /col2: track 157.8 -> 159.9 mm
- net Net-(D10-A): track 5.05 -> 3.09 mm
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