File: main.kicad_sch (KiCad schematic)
At the start: 89 parts, among them SW1 SW_PUSH, SW10 SW_PUSH, SW11 SW_PUSH, SW12 SW_PUSH, SW13 SW_PUSH, SW14 SW_PUSH, SW15 SW_PUSH, SW16 SW_PUSH, SW17 SW_PUSH, SW18 SW_PUSH, SW19 SW_PUSH, SW2 SW_PUSH, SW20 SW_PUSH, SW21 SW_PUSH, SW22 SW_PUSH, SW23 SW_PUSH, SW24 SW_PUSH, SW25 SW_PUSH, SW26 SW_PUSH, SW27 SW_PUSH, SW28 SW_PUSH, SW29 SW_PUSH, SW3 SW_PUSH, SW30 SW_PUSH, SW31 SW_PUSH, SW32 SW_PUSH, SW33 SW_PUSH, SW34 SW_PUSH, SW35 SW_PUSH, SW36 SW_PUSH, SW37 SW_PUSH, SW38 SW_PUSH, SW39 SW_PUSH, SW4 SW_PUSH, SW40 SW_PUSH, SW41 SW_PUSH, SW42 SW_PUSH, SW43 SW_PUSH, SW44 SW_PUSH, SW5 SW_PUSH, SW6 SW_PUSH, SW7 SW_PUSH, SW8 SW_PUSH, SW9 SW_PUSH, U1 RP2040_ZERO

Commit message: :sparkles: (v1) Done. Pre-Order Final Review
Connections:
- net col10: now also U1.6 (GP5); no longer U1.2 (GP1)
- net col11: now also U1.5 (GP4); no longer U1.1 (GP0)
- net col6: now also U1.10 (GP9); no longer U1.6 (GP5)
- net col7: now also U1.9 (GP8); no longer U1.5 (GP4)
- net col8: now also U1.8 (GP7); no longer U1.4 (GP3)
- net col9: now also U1.7 (GP6); no longer U1.3 (GP2)
- net row0: now also U1.4 (GP3); no longer U1.10 (GP9)
- net row1: now also U1.3 (GP2); no longer U1.11 (GP10)
- net row2: now also U1.2 (GP1); no longer U1.12 (GP11)
- net row3: now also U1.1 (GP0); no longer U1.13 (GP12)
Changed lines of the file:
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@@
 	)
 	(no_connect
-		(at 76.2 40.64)
+		(at 52.07 53.34)
 	)
 	(no_connect
-		(at 76.2 43.18)
+		(at 54.61 53.34)
 	)
 	(no_connect
-		(at 76.2 45.72)
+		(at 57.15 53.34)
 	)
 	(no_connect
@@
 		)
 	)
-	(label "col7"
-		(at 76.2 35.56 0)
-		(fields_autoplaced yes)
-		(effects
-			(font
-				(size 1.27 1.27)
-			)
-			(justify left bottom)
-		)
-	)
 	(label "col3"
 		(at 33.02 40.64 180)
@@
 		)
 	)
-	(label "col9"
-		(at 76.2 30.48 0)
-		(fields_autoplaced yes)
-		(effects
-			(font
-				(size 1.27 1.27)
-			)
-			(justify left bottom)
-		)
-	)
-	(label "col8"
-		(at 76.2 33.02 0)
+	(label "col7"
+		(at 76.2 45.72 0)
 		(fields_autoplaced yes)
 		(effects
@@
 	)
 	(label "col11"
-		(at 76.2 25.4 0)
+		(at 76.2 35.56 0)
 		(fields_autoplaced yes)
 		(effects
@@
 		)
 	)
+	(label "row0"
+		(at 76.2 33.02 0)
+		(fields_autoplaced yes)
+		(effects
+			(font
+				(size 1.27 1.27)
+			)
+			(justify left bottom)
+		)
+	)
 	(label "col0"
 		(at 63.5 68.58 90)
@@
 		)
 	)
-	(label "row3"
-		(at 52.07 53.34 270)
-		(fields_autoplaced yes)
-		(effects
-			(font
-				(size 1.27 1.27)
-			)
-			(justify right bottom)
+	(label "col8"
+		(at 76.2 43.18 0)
+		(fields_autoplaced yes)
+		(effects
+			(font
+				(size 1.27 1.27)
+			)
+			(justify left bottom)
+		)
+	)
+	(label "col9"
+		(at 76.2 40.64 0)
+		(fields_autoplaced yes)
+		(effects
+			(font
+				(size 1.27 1.27)
+			)
+			(justify left bottom)
 		)
 	)
@@
 		)
 	)
-	(label "col6"
-		(at 76.2 38.1 0)
-		(fields_autoplaced yes)
-		(effects
-			(font
-				(size 1.27 1.27)
-			)
-			(justify left bottom)
-		)
-	)
 	(label "col5"
 		(at 171.45 68.58 90)
@@
 		)
 	)
+	(label "col10"
+		(at 76.2 38.1 0)
+		(fields_autoplaced yes)
+		(effects
+			(font
+				(size 1.27 1.27)
+			)
+			(justify left bottom)
+		)
+	)
 	(label "col7"
 		(at 214.63 68.58 90)
@@
 		)
 	)
-	(label "row1"
-		(at 57.15 53.34 270)
+	(label "row2"
+		(at 76.2 27.94 0)
+		(fields_autoplaced yes)
+		(effects
+			(font
+				(size 1.27 1.27)
+			)
+			(justify left bottom)
+		)
+	)
+	(label "col6"
+		(at 59.69 53.34 270)
 		(fields_autoplaced yes)
 		(effects
@@
 			)
 			(justify right bottom)
-		)
-	)
-	(label "row2"
-		(at 54.61 53.34 270)
-		(fields_autoplaced yes)
-		(effects
-			(font
-				(size 1.27 1.27)
-			)
-			(justify right bottom)
-		)
-	)
-	(label "col10"
-		(at 76.2 27.94 0)
-		(fields_autoplaced yes)
-		(effects
-			(font
-				(size 1.27 1.27)
-			)
-			(justify left bottom)
 		)
 	)
@@
 		)
 	)
+	(label "row1"
+		(at 76.2 30.48 0)
+		(fields_autoplaced yes)
+		(effects
+			(font
+				(size 1.27 1.27)
+			)
+			(justify left bottom)
+		)
+	)
 	(label "col1"
 		(at 33.02 35.56 180)
@@
 		)
 	)
+	(label "row3"
+		(at 76.2 25.4 0)
+		(fields_autoplaced yes)
+		(effects
+			(font
+				(size 1.27 1.27)
+			)
+			(justify left bottom)
+		)
+	)
 	(label "col6"
 		(at 193.04 68.58 90)
@@
 		(fields_autoplaced yes)
 		(effects
-			(font
-				(size 1.27 1.27)
-			)
-			(justify right bottom)
-		)
-	)
-	(label "row0"
-		(at 59.69 53.34 270)
-		(fields_autoplaced yes)
-		(effects

Commit message: :sparkles: (fix)
Parts:
- added L1, L10, L11, L12, L13, L14, L15, L16, L17, L18, L19, L2, L20, L21, L22, L23, L24, L25, L26, L27, L28, L29, L3, L30, L31, L32, L33, L34, L35, L36, L37, L38, L39, L4, L40, L41, L42, L43, L44, L5, L6, L7, L8, L9: SK6812MINI-E, kamo3_footprint:YS-SK6812MINI-E, symbol kamo3_symbol:SK6812MINI-E
- added Q1: BSS138, Package_TO_SOT_SMD:SOT-23, symbol Transistor_FET:BSS138
- added R1, R2: 10K, Resistor_SMD:R_1206_3216Metric_Pad1.30x1.75mm_HandSolder, symbol Device:R
Connections:
- net +3.3V: now also Q1.1 (G), R1.1
- net GND: now also L1.3 (GND), L10.3 (GND), L11.3 (GND), L12.3 (GND), L13.3 (GND), L14.3 (GND), L15.3 (GND), L16.3 (GND), L17.3 (GND), L18.3 (GND), L19.3 (GND), L2.3 (GND), L20.3 (GND), L21.3 (GND), L22.3 (GND), L23.3 (GND), L24.3 (GND), L25.3 (GND), L26.3 (GND), L27.3 (GND), L28.3 (GND), L29.3 (GND), L3.3 (GND), L30.3 (GND), L31.3 (GND), L32.3 (GND), L33.3 (GND), L34.3 (GND), L35.3 (GND), L36.3 (GND), L37.3 (GND), L38.3 (GND), L39.3 (GND), L4.3 (GND), L40.3 (GND), L41.3 (GND), L42.3 (GND), L43.3 (GND), L44.3 (GND), L5.3 (GND), L6.3 (GND), L7.3 (GND), L8.3 (GND), L9.3 (GND)
- net VDC: now also L1.1 (VDD), L10.1 (VDD), L11.1 (VDD), L12.1 (VDD), L13.1 (VDD), L14.1 (VDD), L15.1 (VDD), L16.1 (VDD), L17.1 (VDD), L18.1 (VDD), L19.1 (VDD), L2.1 (VDD), L20.1 (VDD), L21.1 (VDD), L22.1 (VDD), L23.1 (VDD), L24.1 (VDD), L25.1 (VDD), L26.1 (VDD), L27.1 (VDD), L28.1 (VDD), L29.1 (VDD), L3.1 (VDD), L30.1 (VDD), L31.1 (VDD), L32.1 (VDD), L33.1 (VDD), L34.1 (VDD), L35.1 (VDD), L36.1 (VDD), L37.1 (VDD), L38.1 (VDD), L39.1 (VDD), L4.1 (VDD), L40.1 (VDD), L41.1 (VDD), L42.1 (VDD), L43.1 (VDD), L44.1 (VDD), L5.1 (VDD), L6.1 (VDD), L7.1 (VDD), L8.1 (VDD), L9.1 (VDD), R2.1
- net col0: now also U1.19 (GP28); no longer U1.20 (GP29)
- net col1: now also U1.18 (GP27); no longer U1.19 (GP28)
- net col2: now also U1.11 (GP10); no longer U1.18 (GP27)
- net col3: now also U1.12 (GP11); no longer U1.17 (GP26)
- net col4: now also U1.13 (GP12); no longer U1.16 (GP15)
- net col5: now also U1.14 (GP13); no longer U1.15 (GP14)
- net col6: now also U1.7 (GP6); no longer U1.10 (GP9)
- net col7: now also U1.8 (GP7); no longer U1.9 (GP8)
- net col8: now also U1.9 (GP8); no longer U1.8 (GP7)
- net col9: now also U1.10 (GP9); no longer U1.7 (GP6)
- new net: L1.2 (DOUT), L2.4 (DIN)
- new net: L14.2 (DOUT), L15.4 (DIN)
- new net: L13.2 (DOUT), L14.4 (DIN)
- new net: L40.2 (DOUT), L41.4 (DIN)
- new net: L39.2 (DOUT), L40.4 (DIN)
- new net: L10.4 (DIN), L9.2 (DOUT)
- new net: L8.2 (DOUT), L9.4 (DIN)
- new net: L11.2 (DOUT), L12.4 (DIN)
- new net: L10.2 (DOUT), L11.4 (DIN)
- new net: L4.2 (DOUT), L5.4 (DIN)
- new net: L3.2 (DOUT), L4.4 (DIN)
- new net: L33.2 (DOUT), L34.4 (DIN)
- new net: L32.2 (DOUT), L33.4 (DIN)
- new net: L37.2 (DOUT), L38.4 (DIN)
- new net: L36.2 (DOUT), L37.4 (DIN)
- new net: L2.2 (DOUT), L3.4 (DIN)
- new net: L31.2 (DOUT), L32.4 (DIN)
- new net: L30.2 (DOUT), L31.4 (DIN)
- new net: L12.2 (DOUT), L13.4 (DIN)
- new net: L7.2 (DOUT), L8.4 (DIN)
- new net: L6.2 (DOUT), L7.4 (DIN)
- new net: L27.2 (DOUT), L28.4 (DIN)
- new net: L26.2 (DOUT), L27.4 (DIN)
- new net: L16.2 (DOUT), L17.4 (DIN)
- new net: L15.2 (DOUT), L16.4 (DIN)
- new net: L23.2 (DOUT), L24.4 (DIN)
- new net: L22.2 (DOUT), L23.4 (DIN)
- new net: L20.2 (DOUT), L21.4 (DIN)
- new net: L19.2 (DOUT), L20.4 (DIN)
- new net: L21.2 (DOUT), L22.4 (DIN)
- new net: L35.2 (DOUT), L36.4 (DIN)
- new net: L38.2 (DOUT), L39.4 (DIN)
- new net: L25.2 (DOUT), L26.4 (DIN)
- new net: L24.2 (DOUT), L25.4 (DIN)
- new net: L5.2 (DOUT), L6.4 (DIN)
- new net: L41.2 (DOUT), L42.4 (DIN)
- new net: L18.2 (DOUT), L19.4 (DIN)
- new net: L17.2 (DOUT), L18.4 (DIN)
- new net: L43.2 (DOUT), L44.4 (DIN)
- new net: L42.2 (DOUT), L43.4 (DIN)
- new net: L34.2 (DOUT), L35.4 (DIN)
- new net: L29.2 (DOUT), L30.4 (DIN)
- new net: L28.2 (DOUT), L29.4 (DIN)
- new net led_v3.3: Q1.2 (S), R1.2, U1.20 (GP29)
- new net led_v5: L1.4 (DIN), Q1.3 (D), R2.2
