File: top.kicad_pcb (KiCad board)
At the start: 2 copper layers, 277.7 x 106.4 mm, 44 parts

Commit message: :sparkles: (fix)
Parts:
- moved REF** 8.63 mm to (185.2, 34.8)
- moved REF** 8.63 mm to (222.4, 26.9)
- moved REF** 8.63 mm to (244.3, 23.4)
- moved REF** 8.63 mm to (203.8, 30.8)
- moved REF** 8.54 mm to (166.7, 38.7)
- moved REF** 8.50 mm to (263.3, 25.4)
- moved REF** 5.92 mm to (128.6, 96.7)
- moved REF** 5.82 mm to (91.5, 88.8)
- moved REF** 5.73 mm to (167.3, 96.8)
- moved REF** 5.73 mm to (223.1, 85.0)
- moved REF** 5.73 mm to (185.9, 92.9)
- moved REF** 5.73 mm to (204.5, 88.9)
- moved REF** 5.72 mm to (72.9, 84.8)
- moved REF** 5.68 mm to (110.2, 92.8)
- moved REF** 3.70 mm to (263.3, 63.4)
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
Commit message: update
Parts:
- moved REF** 1.04 mm to (205.2, 69.4)
Changed lines of the file:
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@@
 	(footprint "kamo3_footprint:SW_CherryMX_Topplate_Hole"
 		(layer "F.Cu")
-		(at 206.2 69.1 12)
+		(at 205.2 69.4 12)
 		(property "Reference" "REF**"
 			(at 0 -0.5 12)
